File: Hardware/Cell manager board/Open source BMS SameConn.sch (KiCad schematic (older format))
At the start: 50 parts, among them P1 CONN_01X07, P2 EXT-TMP, P3 CONN_01X09, P4 CONN_01X10, Q1 BSS138, Q2 BSS138, Q3 BSS138, Q4 BSS138, Q5 BSS138, Q6 BSS138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

Commit message: progress
Mostly put together but missing traces
Parts:
- removed 100nF7: Cap, Capacitors_SMD:C_0603, symbol Cap
- removed P4: CONN_01X10, Connectors_Molex:Connector_Molex_PicoBlade_53261-1071, symbol CONN_01X10
- removed R18, R19, R20: 1K, Resistors_SMD:R_Cat16-4, symbol R_PACK4
- added P4: CONN_01X09, Connectors_Molex:Connector_Molex_PicoBlade_53261-0971, symbol CONN_01X09
- added R18, R19, R20, R21, R22, R23, R24: 1KΩ, Resistors_SMD:R_0603, symbol R
Connections:
- net +3.3V: now also P4.2 (P2)
- net GND: now also P4.1 (P1); no longer 100nF6.2, U1.10 (MBAT1)
- net DISCH6: now reaches Q1.1 (G)
- net DISCH6: now also U1.47 (DISCH6)
- net at P1.6 (P6), Q1.2 (S), R7.1: now also D2.1 (A), R19.2; no longer R2.2
- net at Q1.3 (D), R10.2: now also R1.1; no longer D1.2 (K)
- net DISCH5: now reaches U1.1 (DISCH5)
- net DISCH5: now also Q2.1 (G)
- net at U1.11 (IRQ): now also P4.4 (P4)
- net at U1.12 (CLK): now also P4.5 (P5)
- net at U1.13 (CS_N): now also P4.6 (P6)
- net at U1.14 (SCK): now also P4.7 (P7)
- net at U1.15 (MOSI): now also P4.8 (P8)
- net at U1.16 (MISO): now also P4.9 (P9)
- net at 100nF2.2, 100nF3.1, U1.2 (MBAT5): now also R20.1
- net DISCH4: now reaches U1.3 (DISCH4)
- net DISCH4: now also Q3.1 (G)
- net at U1.35 (PD_N_LOW_OUT): now also P4.3 (P3)
- net at 100nF3.2, 100nF4.1, U1.4 (MBAT4): now also R21.1
- net at 100nF1.1, U1.46 (MBAT7): now also R18.1
- net at 100nF1.2, 100nF2.1, U1.48 (MBAT6): now also R19.1
- net DISCH3: now reaches U1.5 (DISCH3)
- net DISCH3: now also Q4.1 (G)
- net at 100nF4.2, 100nF5.1, U1.6 (MBAT3): now also R22.1
- net DISCH2: now reaches U1.7 (DISCH2)
- net DISCH2: now also Q5.1 (G)
- net at 100nF5.2, 100nF6.1, U1.8 (MBAT2): now also R23.1
- net DISCH1: now reaches U1.9 (DISCH1)
- net DISCH1: now also Q6.1 (G)
- net at P1.5 (P5), Q2.2 (S), R8.1: now also D3.1 (A), R20.2; no longer R3.2
- net at P1.4 (P4), Q3.2 (S), R9.1: now also D4.1 (A), R21.2; no longer R4.2
- net at D1.1 (A): now also P1.7 (P7), R10.1, R13.2, R18.2; no longer R1.1
- net at P1.1 (P1), Q6.2 (S), R14.2: now also R24.2
- net at P1.2 (P2), Q5.2 (S), R12.1: now also D6.1 (A), R23.2; no longer R6.2
- net at P1.3 (P3), Q4.2 (S), R11.1: now also D5.1 (A), R22.2; no longer R5.2
- net at R2.1: now also Q2.3 (D), R7.2; no longer D2.1 (A)
- net at Q3.3 (D), R8.2: now also R3.1; no longer D3.2 (K)
- net at Q6.3 (D), R12.2: now also R6.1; no longer D6.2 (K)
- net at Q4.3 (D), R9.2: now also R4.1; no longer D4.2 (K)
- net at Q5.3 (D), R11.2: now also R5.1; no longer D5.2 (K)
- new net: 100nF6.2, R24.1, U1.10 (MBAT1)
- new net: D1.2 (K), R1.2
- new net: D2.2 (K), R2.2
- new net: D3.2 (K), R3.2
- new net: D6.2 (K), R6.2
- new net: D4.2 (K), R4.2
- new net: D5.2 (K), R5.2
Other:
- note removed: "Connectors different so modules can't be wired up backwards. \nThis add a slight but negliagable complexity to constructing cables to go between boards. \nPlus it is much neater to use 10 wire ribbon cables this way."
- moved on the sheet: 100nF1, 100nF2, 100nF3, 100nF4, 100nF5, 100nF6, 100nF9, 10uF1, 33uF1, D1, D2, D3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
