File: Hardware/Cell manager board/Open source BMS.sch (KiCad schematic (older format))
At the start: 50 parts, among them P1 CONN_01X07, P2 EXT-TMP, P3 CONN_01X09, P4 CONN_01X10, Q1 BSS138, Q2 BSS138, Q3 BSS138, Q4 BSS138, Q5 BSS138, Q6 BSS138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

Commit message: progress
Mostly put together but missing traces
Parts:
- 100nF8: footprint (none) -> Capacitors_SMD:C_0603
- 10uF1: footprint (none) -> Capacitors_SMD:C_2220
- 33uF1: footprint (none) -> Capacitors_Tantalum_SMD:TantalC_SizeA_EIA-3216_Reflow
- P2: footprint (none) -> Pin_Headers:Pin_Header_Angled_1x02
- R18: renamed from 1KΩ1; value R_PACK4 -> 1K
- R19: renamed from 1KΩ2; value R_PACK4 -> 1K
- R20: renamed from 1KΩ3; value R_PACK4 -> 1K
Connections:
- net at U1.11 (IRQ): now also P4.5 (P5); no longer P4.10 (P10)
- net at U1.12 (CLK): now also P4.6 (P6); no longer P4.9 (P9)
- net at U1.13 (CS_N): now also P4.7 (P7); no longer P4.8 (P8)
- net at U1.14 (SCK): now also P4.8 (P8); no longer P4.7 (P7)
- net at U1.15 (MOSI): now also P4.9 (P9); no longer P4.6 (P6)
- net at U1.16 (MISO): now also P4.10 (P10); no longer P4.5 (P5)
- net at U1.39 (MISO_IN): now also P3.1 (P1); no longer P3.6 (P6)
- net at U1.40 (MOSI_OUT): now also P3.2 (P2); no longer P3.5 (P5)
- net at U1.41 (SCK_OUT): now also P3.3 (P3); no longer P3.4 (P4)
- net at U1.42 (CS_N_OUT): now also P3.4 (P4); no longer P3.3 (P3)
- net at U1.43 (CLK_OUT): now also P3.5 (P5); no longer P3.2 (P2)
- net at U1.44 (IRQ_IN_): now also P3.6 (P6); no longer P3.1 (P1)
Changed lines of the file:
@@
 $EndComp
 $Comp
-L R_PACK4 1KΩ2
+L R_PACK4 R19
 U 1 1 54154DCE
 P 4400 3150
-F 0 "1KΩ2" H 4400 3600 40  0000 C CNN
-F 1 "R_PACK4" H 4400 3100 40  0000 C CNN
+F 0 "R19" H 4400 3600 40  0000 C CNN
+F 1 "1K" H 4400 3100 40  0000 C CNN
 F 2 "Resistors_SMD:R_Cat16-4" H 4400 3150 60  0000 C CNN
 F 3 "" H 4400 3150 60  0000 C CNN
@@
 $EndComp
 $Comp
-L +BATT #PWR2
+L +BATT #PWR01
 U 1 1 54188DB8
 P 5550 1050
-F 0 "#PWR2" H 5550 1000 20  0001 C CNN
+F 0 "#PWR01" H 5550 1000 20  0001 C CNN
 F 1 "+BATT" H 5550 1150 30  0000 C CNN
 F 2 "" H 5550 1050 60  0000 C CNN
@@
 $EndComp
 $Comp
-L GND #PWR5
+L GND #PWR02
 U 1 1 54188E78
 P 7750 5650
-F 0 "#PWR5" H 7750 5650 30  0001 C CNN
+F 0 "#PWR02" H 7750 5650 30  0001 C CNN
 F 1 "GND" H 7750 5580 30  0001 C CNN
 F 2 "" H 7750 5650 60  0000 C CNN
@@
 To Battery
 $Comp
-L GND #PWR1
+L GND #PWR03
 U 1 1 54237CBF
 P 5150 5050
-F 0 "#PWR1" H 5150 5050 30  0001 C CNN
+F 0 "#PWR03" H 5150 5050 30  0001 C CNN
 F 1 "GND" H 5150 4980 30  0001 C CNN
 F 2 "" H 5150 5050 60  0000 C CNN
@@
 $EndComp
 $Comp
-L R_PACK4 1KΩ1
+L R_PACK4 R18
 U 1 1 54245CCF
 P 4400 2000
-F 0 "1KΩ1" H 4400 2450 40  0000 C CNN
-F 1 "R_PACK4" H 4400 1950 40  0000 C CNN
+F 0 "R18" H 4400 2450 40  0000 C CNN
+F 1 "1K" H 4400 1950 40  0000 C CNN
 F 2 "Resistors_SMD:R_Cat16-4" H 4400 2000 60  0000 C CNN
 F 3 "" H 4400 2000 60  0000 C CNN
@@
 $EndComp
 $Comp
-L R_PACK4 1KΩ3
+L R_PACK4 R20
 U 1 1 54248379
 P 4400 4400
-F 0 "1KΩ3" H 4400 4850 40  0000 C CNN
-F 1 "R_PACK4" H 4400 4350 40  0000 C CNN
+F 0 "R20" H 4400 4850 40  0000 C CNN
+F 1 "1K" H 4400 4350 40  0000 C CNN
 F 2 "Resistors_SMD:R_Cat16-4" H 4400 4400 60  0000 C CNN
 F 3 "" H 4400 4400 60  0000 C CNN
@@
 F 0 "P2" H 5800 4800 50  0000 C CNN
 F 1 "EXT-TMP" V 5900 4650 50  0000 C CNN
-F 2 "" H 5800 4650 60  0000 C CNN
+F 2 "Pin_Headers:Pin_Header_Angled_1x02" H 5800 4650 60  0000 C CNN
 F 3 "" H 5800 4650 60  0000 C CNN
 	1    5800 4650
@@
 $EndComp
 $Comp
-L +BATT #PWR3
+L +BATT #PWR04
 U 1 1 54265091
 P 6100 1050
-F 0 "#PWR3" H 6100 1000 20  0001 C CNN
+F 0 "#PWR04" H 6100 1000 20  0001 C CNN
 F 1 "+BATT" H 6100 1150 30  0000 C CNN
 F 2 "" H 6100 1050 60  0000 C CNN
@@
 $EndComp
 $Comp
-L GND #PWR4
+L GND #PWR05
 U 1 1 54268087
 P 6100 1650
-F 0 "#PWR4" H 6100 1650 30  0001 C CNN
+F 0 "#PWR05" H 6100 1650 30  0001 C CNN
 F 1 "GND" H 6100 1580 30  0001 C CNN
 F 2 "" H 6100 1650 60  0000 C CNN
@@
 F 0 "33uF1" H 10400 4700 40  0000 L CNN
 F 1 "PolC" H 10406 4565 40  0000 L CNN
-F 2 "" H 10438 4500 30  0000 C CNN
+F 2 "Capacitors_Tantalum_SMD:TantalC_SizeA_EIA-3216_Reflow" H 10438 4500 30  0000 C CNN
 F 3 "" H 10250 4600 60  0000 C CNN
 	1    10400 4600
@@
 $EndComp
 $Comp
-L GND #PWR9
+L GND #PWR06
 U 1 1 54255D02
 P 10650 4950
-F 0 "#PWR9" H 10650 4950 30  0001 C CNN
+F 0 "#PWR06" H 10650 4950 30  0001 C CNN
 F 1 "GND" H 10650 4880 30  0001 C CNN
 F 2 "" H 10650 4950 60  0000 C CNN
@@
 $EndComp
 $Comp
-L +BATT #PWR7
+L +BATT #PWR07
 U 1 1 54257090
 P 10650 2850
-F 0 "#PWR7" H 10650 2800 20  0001 C CNN
+F 0 "#PWR07" H 10650 2800 20  0001 C CNN
 F 1 "+BATT" H 10650 2950 30  0000 C CNN
 F 2 "" H 10650 2850 60  0000 C CNN
@@
 F 0 "10uF1" H 6100 1450 40  0000 L CNN
 F 1 "PolC" H 6106 1315 40  0000 L CNN
-F 2 "" H 6138 1250 30  0000 C CNN
+F 2 "Capacitors_SMD:C_2220" H 6138 1250 30  0000 C CNN
 F 3 "" H 5950 1350 60  0000 C CNN
 	1    6100 1350
@@
 F 0 "100nF8" H 8900 5200 40  0000 L CNN
 F 1 "Cap" H 8906 5065 40  0000 L CNN
-F 2 "" H 8938 5000 30  0000 C CNN
+F 2 "Capacitors_SMD:C_0603" H 8938 5000 30  0000 C CNN
 F 3 "" H 8750 5100 60  0000 C CNN
 	1    8900 5100
@@
 Connection ~ 5150 3400
 Wire Wire Line
-	8300 3300 9500 3300
-Wire Wire Line
-	9500 3300 9500 3000
-Wire Wire Line
-	8300 3400 9600 3400
-Wire Wire Line
-	9600 3400 9600 3000
-Wire Wire Line
-	8300 3500 9700 3500
-Wire Wire Line
-	9700 3500 9700 3000
-Wire Wire Line
-	8300 3600 9800 3600
-Wire Wire Line
-	9800 3600 9800 3000
-Wire Wire Line
-	8300 3700 9900 3700
-Wire Wire Line
-	9900 3700 9900 3000
-Wire Wire Line
-	8300 3800 10000 3800
-Wire Wire Line
-	10000 3800 10000 3000
-Wire Wire Line
-	8300 4100 9500 4100
-Wire Wire Line
-	9500 4100 9500 4900
-Wire Wire Line
-	8300 4200 9600 4200
-Wire Wire Line
-	9600 4200 9600 4900
-Wire Wire Line
-	8300 4300 9700 4300
-Wire Wire Line
-	9700 4300 9700 4900
-Wire Wire Line
-	8300 4400 9800 4400
-Wire Wire Line
-	9800 4400 9800 4900
-Wire Wire Line
-	8300 4500 9900 4500
-Wire Wire Line
-	9900 4500 9900 4900
-Wire Wire Line
-	8300 4600 10000 4600
-Wire Wire Line
-	10000 4600 10000 4900
-Wire Wire Line
 	6300 4900 6300 5500
 Wire Wire Line
@@
 	10200 4350 10200 4900
 $Comp
-L GND #PWR6
+L GND #PWR08
 U 1 1 5425E157
 P 8750 5500
-F 0 "#PWR6" H 8750 5500 30  0001 C CNN
+F 0 "#PWR08" H 8750 5500 30  0001 C CNN
 F 1 "GND" H 8750 5430 30  0001 C CNN
 F 2 "" H 8750 5500 60  0000 C CNN
@@
 Connection ~ 8750 5350
 $Comp
-L +3.3V #PWR8
+L +3.3V #PWR09
 U 1 1 54266B58
 P 10650 4250
-F 0 "#PWR8" H 10650 4210 30  0001 C CNN
+F 0 "#PWR09" H 10650 4210 30  0001 C CNN
 F 1 "+3.3V" H 10650 4360 30  0000 C CNN
 F 2 "" H 10650 4250 60  0000 C CNN
@@
 	7250 5500 7250 5400
 Connection ~ 7250 5500
+Wire Wire Line
+	8300 3800 9500 3800
+Wire Wire Line
+	9500 3800 9500 3000
+Wire Wire Line
+	8300 3700 9600 3700
+Wire Wire Line
+	9600 3700 9600 3000
+Wire Wire Line
+	8300 3600 9700 3600
+Wire Wire Line
+	9700 3600 9700 3000
+Wire Wire Line
+	8300 3500 9800 3500
+Wire Wire Line
+	9800 3500 9800 3000
+Wire Wire Line
+	8300 3400 9900 3400
+Wire Wire Line
+	9900 3400 9900 3000
+Wire Wire Line
+	8300 3300 10000 3300
+Wire Wire Line
+	10000 3300 10000 3000
+Wire Wire Line
+	8300 4600 9500 4600
+Wire Wire Line
+	9500 4600 9500 4900
+Wire Wire Line
+	8300 4500 9600 4500
+Wire Wire Line
+	9600 4500 9600 4900
+Wire Wire Line
+	8300 4400 9700 4400
+Wire Wire Line
+	9700 4400 9700 4900
+Wire Wire Line
+	8300 4300 9800 4300
+Wire Wire Line
+	9800 4300 9800 4900
+Wire Wire Line
+	8300 4200 9900 4200
+Wire Wire Line
+	9900 4200 9900 4900
+Wire Wire Line
+	8300 4100 10000 4100
+Wire Wire Line
+	10000 4100 10000 4900
 $EndSCHEMATC

Commit message: board rev1 finished except for silkscreen
bms slave board finished excluding silkscreen
Parts:
- removed 100nF7: Cap, Capacitors_SMD:C_0603, symbol Cap
- removed P4: CONN_01X10, Connectors_Molex:Connector_Molex_PicoBlade_53261-1071, symbol CONN_01X10
- removed R18, R19, R20: 1K, Resistors_SMD:R_Cat16-4, symbol R_PACK4
- added P4: CONN_01X09, MasCustomParts:Connector_SMD_GH_SIDECONN_1X9_1.25MM_45515711ND, symbol CONN_01X09
- added R18, R19, R20, R21, R22, R23, R24: 1KΩ, Resistors_SMD:R_0603, symbol R
- P3: footprint Connectors_Molex:Connector_Molex_PicoBlade_53261-0971 -> MasCustomParts:Connector_SMD_GH_SIDECONN_1X9_1.25MM_45515711ND
Connections:
- net +3.3V: now also P4.2 (P2)
- net GND: now also P4.1 (P1); no longer 100nF6.2, U1.10 (MBAT1)
- net DISCH6: now reaches Q1.1 (G)
- net DISCH6: now also U1.47 (DISCH6)
- net at P1.6 (P6), Q1.2 (S), R7.1: now also D2.1 (A), R19.2; no longer R2.2
- net at Q1.3 (D), R10.2: now also R1.1; no longer D1.2 (K)
- net DISCH5: now reaches U1.1 (DISCH5)
- net DISCH5: now also Q2.1 (G)
- net at U1.11 (IRQ): now also P4.4 (P4)
- net at U1.12 (CLK): now also P4.5 (P5)
- net at U1.13 (CS_N): now also P4.6 (P6)
- net at U1.14 (SCK): now also P4.7 (P7)
- net at U1.15 (MOSI): now also P4.8 (P8)
- net at U1.16 (MISO): now also P4.9 (P9)
- net at 100nF2.2, 100nF3.1, U1.2 (MBAT5): now also R20.1
- net DISCH4: now reaches U1.3 (DISCH4)
- net DISCH4: now also Q3.1 (G)
- net at U1.35 (PD_N_LOW_OUT): now also P4.3 (P3)
- net at 100nF3.2, 100nF4.1, U1.4 (MBAT4): now also R21.1
- net at 100nF1.1, U1.46 (MBAT7): now also R18.1
- net at 100nF1.2, 100nF2.1, U1.48 (MBAT6): now also R19.1
- net DISCH3: now reaches U1.5 (DISCH3)
- net DISCH3: now also Q4.1 (G)
- net at 100nF4.2, 100nF5.1, U1.6 (MBAT3): now also R22.1
- net DISCH2: now reaches U1.7 (DISCH2)
- net DISCH2: now also Q5.1 (G)
- net at 100nF5.2, 100nF6.1, U1.8 (MBAT2): now also R23.1
- net DISCH1: now reaches U1.9 (DISCH1)
- net DISCH1: now also Q6.1 (G)
- net at P1.5 (P5), Q2.2 (S), R8.1: now also D3.1 (A), R20.2; no longer R3.2
- net at P1.4 (P4), Q3.2 (S), R9.1: now also D4.1 (A), R21.2; no longer R4.2
- net at D1.1 (A): now also P1.7 (P7), R10.1, R13.2, R18.2; no longer R1.1
- net at P1.1 (P1), Q6.2 (S), R14.2: now also R24.2
- net at P1.2 (P2), Q5.2 (S), R12.1: now also D6.1 (A), R23.2; no longer R6.2
- net at P1.3 (P3), Q4.2 (S), R11.1: now also D5.1 (A), R22.2; no longer R5.2
- net at R2.1: now also Q2.3 (D), R7.2; no longer D2.1 (A)
- net at Q3.3 (D), R8.2: now also R3.1; no longer D3.2 (K)
- net at Q6.3 (D), R12.2: now also R6.1; no longer D6.2 (K)
- net at Q4.3 (D), R9.2: now also R4.1; no longer D4.2 (K)
- net at Q5.3 (D), R11.2: now also R5.1; no longer D5.2 (K)
- new net: 100nF6.2, R24.1, U1.10 (MBAT1)
- new net: D1.2 (K), R1.2
- new net: D2.2 (K), R2.2
- new net: D3.2 (K), R3.2
- new net: D6.2 (K), R6.2
- new net: D4.2 (K), R4.2
- new net: D5.2 (K), R5.2
Other:
- note removed: "Connectors different so modules can't be wired up backwards. \nThis add a slight but negliagable complexity to constructing cables to go between boards. \nPlus it is much neater to use 10 wire ribbon cables this way."
- moved on the sheet: 100nF1, 100nF2, 100nF3, 100nF4, 100nF5, 100nF6, 100nF9, 10uF1, 33uF1, D1, D2, D3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
