File: Hardware/Cell manager board/Open source BMS.kicad_pcb (KiCad board)
At the start: 2 copper layers, 50 parts, among them P1 CONN_01X07, P2 EXT-TMP, P3 CONN_01X09, P4 CONN_01X10, Q1 BSS138, Q2 BSS138, Q3 BSS138, Q4 BSS138, Q5 BSS138, Q6 BSS138, U1 ATA6870N_BMS

Commit message: board rev1 finished except for silkscreen
bms slave board finished excluding silkscreen
Parts:
- removed 100nF7: Cap, Capacitors_SMD:C_0603
- added R21: 1KΩ, Resistors_SMD:R_0603, F.Cu at (195.7, 126.9)
- added R22: 1KΩ, Resistors_SMD:R_0603, F.Cu at (195.7, 130.0)
- added R23: 1KΩ, Resistors_SMD:R_0603, F.Cu at (195.7, 133.2)
- added R24: 1KΩ, Resistors_SMD:R_0603, F.Cu at (195.7, 136.4)
- P1: footprint Pin_Headers:Pin_Header_Angled_1x07 -> Pin_Header_Angled_1x07
- P3: footprint Connectors_Molex:Connector_Molex_PicoBlade_53261-0971 -> MasCustomParts:Connector_SMD_GH_SIDECONN_1X9_1.25MM_45515711ND
- P4: value CONN_01X10 -> CONN_01X09; footprint Connectors_Molex:Connector_Molex_PicoBlade_53261-1071 -> MasCustomParts:Connector_SMD_GH_SIDECONN_1X9_1.25MM_45515711ND
- Q1, Q2, Q3, Q4, Q5, Q6: footprint SMD_Packages:SOT-23 -> SOT-23
- R10, R11, R12, R7, R8, R9: moved to F.Cu
- R18, R19, R20: value 1K -> 1KΩ; footprint Resistors_SMD:R_Cat16-4 -> Resistors_SMD:R_0603
- moved 10uF1 161.3 mm to (206.2, 119.1)
- moved R16 159.5 mm to (212.1, 130.3), turned to 180 degrees
- moved R14 154.3 mm to (195.7, 141.5), turned to 270 degrees
- moved R15 151.2 mm to (212.1, 131.8), turned to 180 degrees
- moved R13 146.7 mm to (198.9, 115.4), turned to 180 degrees
- moved TH1 134.5 mm to (190.5, 128.8), turned to 90 degrees
- moved R12 118.8 mm to (181.6, 144.8)
- moved R11 118.6 mm to (181.6, 138.4)
- moved R9 118.4 mm to (181.6, 132.1)
- moved R8 118.2 mm to (181.6, 125.7)
- moved R7 118.0 mm to (181.6, 119.4)
- moved R10 117.8 mm to (181.6, 113.0)
- moved Q6 117.6 mm to (189.2, 144.8)
- moved Q5 117.3 mm to (189.2, 138.4)
- moved P1 117.1 mm to (172.7, 130.8)
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Connections:
- 100nF6 pad 2: GND -> Net-(100nF6-Pad2)
- P1 pad 2: Net-(P1-Pad2) -> Net-(D6-Pad1)
- P1 pad 3: Net-(P1-Pad3) -> Net-(D5-Pad1)
- P1 pad 4: Net-(P1-Pad4) -> Net-(D4-Pad1)
- P1 pad 5: Net-(P1-Pad5) -> Net-(D3-Pad1)
- P1 pad 6: Net-(P1-Pad6) -> Net-(D2-Pad1)
- P1 pad 7: Net-(P1-Pad7) -> Net-(D1-Pad1)
- P4 pad 2: Net-(P4-Pad2) -> +3.3V
- P4 pad 3: +3.3V -> Net-(P4-Pad3)
- Q1 pad 1: Net-(Q1-Pad1) -> /DISCH6
- Q1 pad 2: Net-(P1-Pad6) -> Net-(D2-Pad1)
- Q1 pad 3: Net-(D1-Pad2) -> Net-(Q1-Pad3)
- Q2 pad 1: Net-(Q2-Pad1) -> /DISCH5
- Q2 pad 2: Net-(P1-Pad5) -> Net-(D3-Pad1)
- Q2 pad 3: Net-(D2-Pad2) -> Net-(Q2-Pad3)
- Q3 pad 1: Net-(Q3-Pad1) -> /DISCH4
- Q3 pad 2: Net-(P1-Pad4) -> Net-(D4-Pad1)
- Q3 pad 3: Net-(D3-Pad2) -> Net-(Q3-Pad3)
- Q4 pad 1: Net-(Q4-Pad1) -> /DISCH3
- Q4 pad 2: Net-(P1-Pad3) -> Net-(D5-Pad1)
- Q4 pad 3: Net-(D4-Pad2) -> Net-(Q4-Pad3)
- Q5 pad 1: Net-(Q5-Pad1) -> /DISCH2
- Q5 pad 2: Net-(P1-Pad2) -> Net-(D6-Pad1)
- Q5 pad 3: Net-(D5-Pad2) -> Net-(Q5-Pad3)
- Q6 pad 1: Net-(Q6-Pad1) -> /DISCH1
- Q6 pad 3: Net-(D6-Pad2) -> Net-(Q6-Pad3)
- R1 pad 1: Net-(D1-Pad1) -> Net-(Q1-Pad3)
- R1 pad 2: Net-(P1-Pad7) -> Net-(D1-Pad2)
- R10 pad 1: Net-(P1-Pad7) -> Net-(D1-Pad1)
- R10 pad 2: Net-(D1-Pad2) -> Net-(Q1-Pad3)
- R11 pad 1: Net-(P1-Pad3) -> Net-(D5-Pad1)
- R11 pad 2: Net-(D5-Pad2) -> Net-(Q5-Pad3)
- R12 pad 1: Net-(P1-Pad2) -> Net-(D6-Pad1)
- R12 pad 2: Net-(D6-Pad2) -> Net-(Q6-Pad3)
- R13 pad 2: Net-(P1-Pad7) -> Net-(D1-Pad1)
- R18 pad 1: Net-(P1-Pad7) -> Net-(100nF1-Pad1)
- R18 pad 2: Net-(Q1-Pad1) -> Net-(D1-Pad1)
- R19 pad 1: Net-(P1-Pad5) -> Net-(100nF1-Pad2)
- R19 pad 2: Net-(Q3-Pad1) -> Net-(D2-Pad1)
- R2 pad 1: Net-(D2-Pad1) -> Net-(Q2-Pad3)
- R2 pad 2: Net-(P1-Pad6) -> Net-(D2-Pad2)
- R20 pad 1: Net-(P1-Pad3) -> Net-(100nF2-Pad2)
- R20 pad 2: Net-(Q5-Pad1) -> Net-(D3-Pad1)
- R3 pad 1: Net-(D3-Pad1) -> Net-(Q3-Pad3)
- R3 pad 2: Net-(P1-Pad5) -> Net-(D3-Pad2)
- R4 pad 1: Net-(D4-Pad1) -> Net-(Q4-Pad3)
- R4 pad 2: Net-(P1-Pad4) -> Net-(D4-Pad2)
- R5 pad 1: Net-(D5-Pad1) -> Net-(Q5-Pad3)
- R5 pad 2: Net-(P1-Pad3) -> Net-(D5-Pad2)
- R6 pad 1: Net-(D6-Pad1) -> Net-(Q6-Pad3)
- R6 pad 2: Net-(P1-Pad2) -> Net-(D6-Pad2)
- R7 pad 1: Net-(P1-Pad6) -> Net-(D2-Pad1)
- R7 pad 2: Net-(D2-Pad2) -> Net-(Q2-Pad3)
- R8 pad 1: Net-(P1-Pad5) -> Net-(D3-Pad1)
- R8 pad 2: Net-(D3-Pad2) -> Net-(Q3-Pad3)
- R9 pad 1: Net-(P1-Pad4) -> Net-(D4-Pad1)
- R9 pad 2: Net-(D4-Pad2) -> Net-(Q4-Pad3)
- U1 pad 1: Net-(R18-Pad5) -> /DISCH5
- U1 pad 10: GND -> Net-(100nF6-Pad2)
- U1 pad 11: Net-(P4-Pad5) -> Net-(P4-Pad4)
- U1 pad 12: Net-(P4-Pad6) -> Net-(P4-Pad5)
- U1 pad 13: Net-(P4-Pad7) -> Net-(P4-Pad6)
- U1 pad 14: Net-(P4-Pad8) -> Net-(P4-Pad7)
- U1 pad 15: Net-(P4-Pad9) -> Net-(P4-Pad8)
- U1 pad 16: Net-(P4-Pad10) -> Net-(P4-Pad9)
- U1 pad 3: Net-(R19-Pad7) -> /DISCH4
- U1 pad 35: Net-(P4-Pad4) -> Net-(P4-Pad3)
- U1 pad 47: Net-(R18-Pad7) -> /DISCH6
- U1 pad 5: Net-(R19-Pad5) -> /DISCH3
- U1 pad 7: Net-(R20-Pad7) -> /DISCH2
- U1 pad 9: Net-(R20-Pad5) -> /DISCH1
Routing:
- net GND: track 0.00 -> 143.1 mm, vias 0 -> 16
- net Net-(P2-Pad2): track 0.00 -> 62.9 mm
- net Net-(D6-Pad1): track 0.00 -> 61.5 mm, vias 0 -> 1
- net Net-(D2-Pad1): track 0.00 -> 55.2 mm, vias 0 -> 1
- net Net-(D5-Pad1): track 0.00 -> 55.0 mm, vias 0 -> 1
- net Net-(D3-Pad1): track 0.00 -> 52.2 mm, vias 0 -> 1
- net Net-(D4-Pad1): track 0.00 -> 51.8 mm, vias 0 -> 1
- net Net-(Q6-Pad3): track 0.00 -> 51.5 mm, vias 0 -> 12
- net Net-(Q5-Pad3): track 0.00 -> 51.0 mm, vias 0 -> 12
- net Net-(D1-Pad1): track 0.00 -> 50.1 mm
- net Net-(P1-Pad1): track 0.00 -> 49.5 mm
- net Net-(Q4-Pad3): track 0.00 -> 47.9 mm, vias 0 -> 12
- net Net-(R16-Pad2): track 0.00 -> 43.4 mm, vias 0 -> 2
- net Net-(Q3-Pad3): track 0.00 -> 42.8 mm, vias 0 -> 12
- net +3.3V: track 0.00 -> 39.5 mm, vias 0 -> 2
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- added copper zone on B.Cu, net GND
- added copper zone on F.Cu, net GND
- added copper zone on B.Cu, net Net-(Q1-Pad3)
- added copper zone on F.Cu, net Net-(Q1-Pad3)
- added copper zone on B.Cu, net Net-(Q2-Pad3)
- added copper zone on F.Cu, net Net-(Q2-Pad3)
- added copper zone on B.Cu, net Net-(Q3-Pad3)
- added copper zone on F.Cu, net Net-(Q3-Pad3)
- added copper zone on B.Cu, net Net-(Q4-Pad3)
- added copper zone on F.Cu, net Net-(Q4-Pad3)
- added copper zone on B.Cu, net Net-(Q5-Pad3)
- added copper zone on F.Cu, net Net-(Q5-Pad3)
- added copper zone on B.Cu, net Net-(Q6-Pad3)
- added copper zone on F.Cu, net Net-(Q6-Pad3)
Other:
- board outline added: 49 x 49 mm
- net class Default: clearance 0.254 -> 0.2032
- rule trace_clearance: 0.254 -> 0.2032
- rule trace_min: 0.254 -> 0.1524
- rule via_min_drill: 0.508 -> 0.3302
- rule via_min_size: 0.889 -> 0.508

Commit message: forgot stuff
ditto
Routing:
- net Net-(Q1-Pad3): vias 12 -> 11
Changed lines of the file:
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@@
     (links 119)
     (no_connects 0)
-    (area 162.281799 103.2718 215.153915 155.6082)
+    (area 165.949999 104.949999 215.050001 154.050001)
     (thickness 1.6)
     (drawings 4)
-    (tracks 739)
+    (tracks 741)
     (zones 0)
     (modules 53)
@@
   )
   (layers
-    (0 F.Cu signal)
-    (31 B.Cu signal)
-    (32 B.Adhes user)
-    (33 F.Adhes user)
+    (0 F.Cu signal hide)
+    (31 B.Cu signal hide)
+    (32 B.Adhes user hide)
+    (33 F.Adhes user hide)
     (34 B.Paste user)
     (35 F.Paste user)
@@
     (38 B.Mask user)
     (39 F.Mask user)
-    (40 Dwgs.User user)
-    (41 Cmts.User user)
-    (42 Eco1.User user)
-    (43 Eco2.User user)
-    (44 Edge.Cuts user)
-    (45 Margin user)
-    (46 B.CrtYd user)
-    (47 F.CrtYd user)
-    (48 B.Fab user)
-    (49 F.Fab user)
+    (40 Dwgs.User user hide)
+    (41 Cmts.User user hide)
+    (42 Eco1.User user hide)
+    (43 Eco2.User user hide)
+    (44 Edge.Cuts user hide)
+    (45 Margin user hide)
+    (46 B.CrtYd user hide)
+    (47 F.CrtYd user hide)
+    (48 B.Fab user hide)
+    (49 F.Fab user hide)
   )
   (setup
-    (last_trace_width 0.4064)
+    (last_trace_width 0.254)
     (user_trace_width 0.1524)
     (user_trace_width 0.2032)
@@
     (pad_to_mask_clearance 0)
     (aux_axis_origin 0 0)
-    (grid_origin 165.862 154.178)
-    (visible_elements 7FFCDF79)
+    (grid_origin 176.2394 111.0002)
+    (visible_elements 7FFFC001)
     (pcbplotparams
       (layerselection 0x00030_80000001)
@@
       (effects (font (size 1.27 1.27) (thickness 0.2032)))
     )
-    (fp_text value CONN_01X07 (at 0 0 90) (layer F.SilkS) hide
+    (fp_text value CONN_01X07 (at 0.7598 -2.8306 90) (layer F.SilkS) hide
       (effects (font (size 1.27 1.27) (thickness 0.2032)))
     )
@@
       (effects (font (size 1.27 1.27) (thickness 0.2032)))
     )
-    (fp_text value EXT-TMP (at 0 0 90) (layer F.SilkS) hide
+    (fp_text value EXT-TMP (at 0.1248 -2.8306 90) (layer F.SilkS) hide
       (effects (font (size 1.27 1.27) (thickness 0.2032)))
     )
@@
       (effects (font (size 1.5 1.5) (thickness 0.15)))
     )
-    (fp_text value R10 (at -0.9 3.4) (layer F.SilkS)
+    (fp_text value R10 (at -5.3706 3.0502) (layer F.SilkS)
       (effects (font (size 1.5 1.5) (thickness 0.15)))
     )
@@
       (effects (font (size 1.5 1.5) (thickness 0.15)))
     )
-    (fp_text value R10 (at -0.9 3.4) (layer F.SilkS)
+    (fp_text value R10 (at -5.3706 3.0502) (layer F.SilkS) hide
       (effects (font (size 1.5 1.5) (thickness 0.15)))
     )
@@
       (effects (font (size 1.5 1.5) (thickness 0.15)))
     )
-    (fp_text value R10 (at -0.9 3.4) (layer F.SilkS)
+    (fp_text value R10 (at -5.3706 3.0502) (layer F.SilkS)
       (effects (font (size 1.5 1.5) (thickness 0.15)))
     )
@@
       (effects (font (size 1.5 1.5) (thickness 0.15)))
     )
-    (fp_text value 10Ω (at -0.9 3.4) (layer F.SilkS)
+    (fp_text value 10Ω (at -4.7356 3.0502) (layer F.SilkS)
       (effects (font (size 1.5 1.5) (thickness 0.15)))
     )
@@
       (effects (font (size 1.5 1.5) (thickness 0.15)))
     )
-    (fp_text value R10 (at -0.9 3.4) (layer F.SilkS)
+    (fp_text value R10 (at -5.3706 3.0502) (layer F.SilkS)
       (effects (font (size 1.5 1.5) (thickness 0.15)))
     )
@@
       (effects (font (size 1.5 1.5) (thickness 0.15)))
     )
-    (fp_text value R10 (at -0.9 3.4) (layer F.SilkS)
+    (fp_text value R10 (at -2.8306 3.6852) (layer F.SilkS)
       (effects (font (size 1.5 1.5) (thickness 0.15)))
     )
@@
   (segment (start 206.502 140.208) (end 210.312 140.208) (width 0.2032) (layer F.Cu) (net 23))
   (segment (start 204.9907 138.6967) (end 206.502 140.208) (width 0.2032) (layer F.Cu) (net 23))
+  (segment (start 195.695 135.636) (end 195.707 135.648) (width 0.2032) (layer F.Cu) (net 24))
+  (segment (start 194.564 135.636) (end 195.695 135.636) (width 0.2032) (layer F.Cu) (net 24))
+  (segment (start 194.31 135.89) (end 194.564 135.636) (width 0.2032) (layer F.Cu) (net 24))
+  (segment (start 192.786 137.414) (end 194.31 135.89) (width 0.2032) (layer F.Cu) (net 24))
+  (segment (start 192.786 137.414) (end 192.786 142.24) (width 0.2032) (layer F.Cu) (net 24))
+  (segment (start 192.786 136.398) (end 192.786 137.414) (width 0.2032) (layer F.Cu) (net 24))
   (segment (start 195.707 142.228) (end 195.707 142.748) (width 0.254) (layer F.Cu) (net 24))
   (segment (start 190.881 147.574) (end 189.23 147.574) (width 0.254) (layer F.Cu) (net 24))
@@
   (segment (start 176.276 147.066) (end 177.546 148.336) (width 0.508) (layer F.Cu) (net 24))
   (segment (start 189.9285 143.8275) (end 190.32982 143.8275) (width 0.6096) (layer F.Cu) (net 24))
-  (segment (start 195.707 135.648) (end 193.536 135.648) (width 0.2032) (layer F.Cu) (net 24))
-  (segment (start 193.536 135.648) (end 192.786 136.398) (width 0.2032) (layer F.Cu) (net 24))
-  (segment (start 192.786 136.398) (end 192.786 142.24) (width 0.2032) (layer F.Cu) (net 24))
   (segment (start 192.786 142.24) (end 191.1985 143.8275) (width 0.2032) (layer F.Cu) (net 24))
   (segment (start 191.1985 143.8275) (end 190.32982 143.8275) (width 0.2032) (layer F.Cu) (net 24))
@@
   (segment (start 197.866 131.953) (end 196.596 133.223) (width 0.2032) (layer F.Cu) (net 48))
   (segment (start 194.818 133.223) (end 194.691 133.223) (width 0.2032) (layer F.Cu) (net 48))
-  (segment (start 194.818 136.398) (end 193.802 136.398) (width 0.2032) (layer F.Cu) (net 49))
-  (segment (start 193.802 136.398) (end 193.548 136.652) (width 0.2032) (layer F.Cu) (net 49))
-  (segment (start 193.548 136.652) (end 193.548 143.51) (width 0.2032) (layer F.Cu) (net 49))
+  (segment (start 193.548 137.414) (end 193.548 143.51) (width 0.2032) (layer F.Cu) (net 49))
+  (segment (start 194.564 136.398) (end 193.548 137.414) (width 0.2032) (layer F.Cu) (net 49))
+  (segment (start 194.818 136.398) (end 194.564 136.398) (width 0.2032) (layer F.Cu) (net 49))
+  (segment (start 198.12 135.128) (end 197.866 135.128) (width 0.2032) (layer F.Cu) (net 49))
+  (segment (start 201.56678 131.30022) (end 199.8345 133.0325) (width 0.2032) (layer F.Cu) (net 49))
+  (segment (start 202.34148 131.30022) (end 201.56678 131.30022) (width 0.2032) (layer F.Cu) (net 49))
+  (segment (start 199.8345 134.9375) (end 199.644 135.128) (width 0.2032) (layer F.Cu) (net 49))
+  (segment (start 199.644 135.128) (end 198.12 135.128) (width 0.2032) (layer F.Cu) (net 49))
+  (segment (start 199.8345 133.0325) (end 199.8345 134.9375) (width 0.2032) (layer F.Cu) (net 49))
+  (segment (start 196.596 136.398) (end 194.818 136.398) (width 0.2032) (layer F.Cu) (net 49))
+  (segment (start 197.866 135.128) (end 196.596 136.398) (width 0.2032) (layer F.Cu) (net 49))
+  (segment (start 191.3255 145.7325) (end 190.32982 145.7325) (width 0.2032) (layer F.Cu) (net 49))
   (segment (start 193.548 143.51) (end 191.3255 145.7325) (width 0.2032) (layer F.Cu) (net 49))
-  (segment (start 191.3255 145.7325) (end 190.32982 145.7325) (width 0.2032) (layer F.Cu) (net 49))
-  (segment (start 197.866 135.128) (end 196.596 136.398) (width 0.2032) (layer F.Cu) (net 49))
-  (segment (start 196.596 136.398) (end 194.818 136.398) (width 0.2032) (layer F.Cu) (net 49))
-  (segment (start 199.8345 133.0325) (end 199.8345 134.9375) (width 0.2032) (layer F.Cu) (net 49))
-  (segment (start 199.644 135.128) (end 198.12 135.128) (width 0.2032) (layer F.Cu) (net 49))
-  (segment (start 199.8345 134.9375) (end 199.644 135.128) (width 0.2032) (layer F.Cu) (net 49))
-  (segment (start 202.34148 131.30022) (end 201.56678 131.30022) (width 0.2032) (layer F.Cu) (net 49))
-  (segment (start 201.56678 131.30022) (end 199.8345 133.0325) (width 0.2032) (layer F.Cu) (net 49))
-  (segment (start 198.12 135.128) (end 197.866 135.128) (width 0.2032) (layer F.Cu) (net 49))
   (segment (start 174.498 109.855) (end 175.133 109.855) (width 0.254) (layer B.Cu) (net 50))
+  (segment (start 175.133 109.855) (end 178.308 113.03) (width 0.254) (layer B.Cu) (net 50))
+  (segment (start 178.308 113.03) (end 180.34 113.03) (width 0.254) (layer B.Cu) (net 50))
+  (segment (start 173.47 109.855) (end 174.498 109.855) (width 0.254) (layer F.Cu) (net 50))
+  (via (at 174.498 109.855) (size 0.889) (layers F.Cu B.Cu) (net 50))
+  (via (at 180.34 113.03) (size 0.889) (layers F.Cu B.Cu) (net 50))
   (segment (start 180.34 113.03) (end 185.11 113.03) (width 0.4064) (layer F.Cu) (net 50))
-  (via (at 180.34 113.03) (size 0.889) (layers F.Cu B.Cu) (net 50))
-  (segment (start 178.308 113.03) (end 180.34 113.03) (width 0.254) (layer B.Cu) (net 50))
-  (segment (start 175.133 109.855) (end 178.308 113.03) (width 0.254) (layer B.Cu) (net 50))
   (segment (start 180.34 111.506) (end 180.34 111.252) (width 0.254) (layer B.Cu) (net 50))
   (segment (start 180.34 111.506) (end 181.864 111.506) (width 0.4064) (layer F.Cu) (net 50))
@@
   (via (at 183.388 111.506) (size 0.889) (layers F.Cu B.Cu) (net 50))
   (segment (start 181.864 111.506) (end 183.388 111.506) (width 0.4064) (layer F.Cu) (net 50))
-  (via (at 180.34 111.506) (size 0.889) (layers F.Cu B.Cu) (net 50))
-  (via (at 174.498 109.855) (size 0.889) (layers F.Cu B.Cu) (net 50))
-  (segment (start 174.498 109.855) (end 173.47 109.855) (width 0.254) (layer F.Cu) (net 50))
   (segment (start 188.13018 113.03) (end 185.11 113.03) (width 0.4064) (layer F.Cu) (net 50))
   (segment (start 188.13018 114.63782) (end 187.96 114.808) (width 0.4064) (layer F.Cu) (net 50))
