File: Hardware/MicroMaster/OSBMS MicroMaster atmega328.sch (KiCad schematic (older format))
At the start: 31 parts, among them IC1 ATMEGA328P-A, P1 CONN_01X06, P10 CONN_01X04, P2 CONN_02X03, P3 CONN_01X03, P4 CONN_01X03, P5 CONN_01X09, P6 CONN_01X10, P7 CONN_01X06, Q1 FDS6892A, Q2 BSS138

Commit message: work dump
board schematics should be working. may include some unfinished
schematics and software pieces
Parts:
- C5: symbol CP1 -> CP1-RESCUE-OSBMS_MicroMaster_atmega328
- D1: symbol ZENER -> ZENER-RESCUE-OSBMS_MicroMaster_atmega328
- IC1: symbol ATMEGA328P-A -> ATMEGA328P-A-RESCUE-OSBMS_MicroMaster_atmega328
- Q1: symbol FDS6892A -> FDS6892A-RESCUE-OSBMS_MicroMaster_atmega328
- R1, R2, R3, R5, R6, R7, R8, R9: symbol R -> R-RESCUE-OSBMS_MicroMaster_atmega328
Connections:
- net D9*: no longer IC1.13 ((PCINT1/OC1A)PB1)
- net 400khz_clk: now reaches P5.5 (P5)
- net 400khz_clk: now also IC1.13 ((PCINT1/OC1A)PB1)
Changed lines of the file:
@@
 EESchema Schematic File Version 2
+LIBS:OSBMS MicroMaster atmega328-rescue
 LIBS:power
 LIBS:device
@@
 LIBS:memory
 LIBS:xilinx
-LIBS:special
 LIBS:microcontrollers
 LIBS:dsp
@@
 $EndDescr
 $Comp
-L ATMEGA328P-A IC1
+L ATMEGA328P-A-RESCUE-OSBMS_MicroMaster_atmega328 IC1
 U 1 1 5434A70A
 P 2550 2350
@@
 $EndComp
 $Comp
-L +3.3V #PWR01
+L +3.3V-RESCUE-OSBMS_MicroMaster_atmega328 #PWR01
 U 1 1 54358F9D
 P 10000 3300
@@
 $EndComp
 $Comp
-L GND #PWR02
+L GND-RESCUE-OSBMS_MicroMaster_atmega328 #PWR02
 U 1 1 54358FB1
 P 10550 3550
@@
 A7
 $Comp
-L GND #PWR03
+L GND-RESCUE-OSBMS_MicroMaster_atmega328 #PWR03
 U 1 1 543DF112
 P 4850 2050
@@
 $EndComp
 $Comp
-L +3.3V #PWR04
+L +3.3V-RESCUE-OSBMS_MicroMaster_atmega328 #PWR04
 U 1 1 543DF1C2
 P 1550 1150
@@
 $EndComp
 $Comp
-L GND #PWR05
+L GND-RESCUE-OSBMS_MicroMaster_atmega328 #PWR05
 U 1 1 543DFD82
 P 1550 3650
@@
 $EndComp
 $Comp
-L GND #PWR06
+L GND-RESCUE-OSBMS_MicroMaster_atmega328 #PWR06
 U 1 1 543E0940
 P 1550 2250
@@
 Text GLabel 4200 1250 2    60   Input ~ 0
 D8
-Text GLabel 3950 1350 2    60   Input ~ 0
+Text GLabel 4650 1350 2    60   Input ~ 0
 D9*
 Text GLabel 3600 1450 2    60   Input ~ 0
@@
 RXD
 $Comp
-L GND #PWR07
+L GND-RESCUE-OSBMS_MicroMaster_atmega328 #PWR07
 U 1 1 543F748F
 P 10250 1750
@@
 $EndComp
 $Comp
-L +3.3V #PWR08
+L +3.3V-RESCUE-OSBMS_MicroMaster_atmega328 #PWR08
 U 1 1 543F915B
 P 10100 1000
@@
 RESET
 $Comp
-L +3.3V #PWR09
+L +3.3V-RESCUE-OSBMS_MicroMaster_atmega328 #PWR09
 U 1 1 543FA4A0
 P 7800 950
@@
 $EndComp
 $Comp
-L GND #PWR010
+L GND-RESCUE-OSBMS_MicroMaster_atmega328 #PWR010
 U 1 1 543FA4C1
 P 7800 1600
@@
 $EndComp
 $Comp
-L R R1
+L R-RESCUE-OSBMS_MicroMaster_atmega328 R1
 U 1 1 5440DAFF
 P 7450 1050
@@
 $EndComp
 $Comp
-L +3.3V #PWR011
+L +3.3V-RESCUE-OSBMS_MicroMaster_atmega328 #PWR011
 U 1 1 545F0369
 P 7750 2250
@@
 $EndComp
 $Comp
-L GND #PWR012
+L GND-RESCUE-OSBMS_MicroMaster_atmega328 #PWR012
 U 1 1 545F036F
 P 7850 3100
@@
 $EndComp
 $Comp
-L +3.3V #PWR013
+L +3.3V-RESCUE-OSBMS_MicroMaster_atmega328 #PWR013
 U 1 1 545F0FA0
 P 9550 5050
@@
 CS_N
 $Comp
-L FDS6892A Q1
+L FDS6892A-RESCUE-OSBMS_MicroMaster_atmega328 Q1
 U 1 1 5464D242
 P 1500 6950
@@
 $EndComp
 $Comp
-L FDS6892A Q1
+L FDS6892A-RESCUE-OSBMS_MicroMaster_atmega328 Q1
 U 2 1 5464D249
 P 2650 7150
@@
 D6*
 $Comp
-L R R9
+L R-RESCUE-OSBMS_MicroMaster_atmega328 R9
 U 1 1 5464D25B
 P 2450 7400
@@
 $EndComp
 $Comp
-L R R7
+L R-RESCUE-OSBMS_MicroMaster_atmega328 R7
 U 1 1 5464D262
 P 1300 7200
@@
 $EndComp
 $Comp
-L GND #PWR014
+L GND-RESCUE-OSBMS_MicroMaster_atmega328 #PWR014
 U 1 1 5464D273
 P 1600 7300
@@
 $EndComp
 $Comp
-L GND #PWR015
+L GND-RESCUE-OSBMS_MicroMaster_atmega328 #PWR015
 U 1 1 5464D279
 P 2750 7500
@@
 $EndComp
 $Comp
-L GND #PWR016
+L GND-RESCUE-OSBMS_MicroMaster_atmega328 #PWR016
 U 1 1 5464D297
 P 5450 7550
@@
 A0
 $Comp
-L R R6
+L R-RESCUE-OSBMS_MicroMaster_atmega328 R6
 U 1 1 5464D2B2
 P 1700 5700
@@
 $EndComp
 $Comp
-L R R5
+L R-RESCUE-OSBMS_MicroMaster_atmega328 R5
 U 1 1 5464D2B9
 P 1700 5100
@@
 $EndComp
 $Comp
-L GND #PWR019
+L GND-RESCUE-OSBMS_MicroMaster_atmega328 #PWR019
 U 1 1 5464D2EC
 P 2100 6100
@@
 Auxilary power outputs\nFor contactor/ETC
 $Comp
-L CP1 C5
+L CP1-RESCUE-OSBMS_MicroMaster_atmega328 C5
 U 1 1 5464D2FB
 P 2100 5450
@@
 D4
 $Comp
-L R R8
+L R-RESCUE-OSBMS_MicroMaster_atmega328 R8
 U 1 1 546576DE
 P 4450 7300
@@
 SDA/A4
 $Comp
-L R R2
+L R-RESCUE-OSBMS_MicroMaster_atmega328 R2
 U 1 1 54692C2B
 P 9850 2350
@@
 $EndComp
 $Comp
-L R R3
+L R-RESCUE-OSBMS_MicroMaster_atmega328 R3
 U 1 1 54692E9E
 P 9850 2500
@@
 $EndComp
 $Comp
-L +3.3V #PWR020
+L +3.3V-RESCUE-OSBMS_MicroMaster_atmega328 #PWR020
 U 1 1 54693308
 P 9550 2300
@@
 D10*
 $Comp
-L GND #PWR021
+L GND-RESCUE-OSBMS_MicroMaster_atmega328 #PWR021
 U 1 1 5469DB42
 P 10650 5350
@@
 $EndComp
 $Comp
-L GND #PWR022
+L GND-RESCUE-OSBMS_MicroMaster_atmega328 #PWR022
 U 1 1 54647FB6
 P 4450 5450
@@
 $EndComp
 $Comp
-L +3.3V #PWR023
+L +3.3V-RESCUE-OSBMS_MicroMaster_atmega328 #PWR023
 U 1 1 54648505
 P 4450 5000
@@
 Connection ~ 3050 6400
 $Comp
-L GND #PWR024
+L GND-RESCUE-OSBMS_MicroMaster_atmega328 #PWR024
 U 1 1 5465EF37
 P 3150 7000
@@
 MOSI
 $Comp
-L ZENER D1
+L ZENER-RESCUE-OSBMS_MicroMaster_atmega328 D1
 U 1 1 54694E07
 P 5250 7100
@@
 Wire Wire Line
 	5250 6800 5250 6900
+Text GLabel 10450 3050 0    60   Input ~ 0
+400khz_clk
+Wire Wire Line
+	10650 3050 10450 3050
+Text GLabel 3950 1350 2    60   Input ~ 0
+400khz_clk
 $EndSCHEMATC
